File: pcb/dev_board.kicad_sch (KiCad schematic)
At the start: 44 parts, among them J1 Conn_02x13_Odd_Even, J2 Conn_02x13_Odd_Even, J4 Conn_01x05, J5 Screw_Terminal_01x03, Q1 Si2356DS, Q2 Si2356DS, Q5 2N3906, Q6 MMBT3904, Q7 MMBT3906, SW1 SW_DIP_x04, U1 XS-LDT-01, U2 MAX5026, U3 KXTJ3-1057, U4 MCP1640BCH, U6 TLV74311

Commit message: V0.2 pcb placement, good enough to proceed/.
Parts:
- removed D1: ES1J, Diode_SMD:D_SMA, symbol Diode:1N4007
- removed Q5: 2N3906, Package_TO_SOT_SMD:SOT-23, symbol Transistor_BJT:2N3906
- removed R2: 10K, Resistor_SMD:R_0603_1608Metric, symbol Device:R
- removed R6: 100K, Resistor_SMD:R_0603_1608Metric, symbol Device:R
- L1: value L_Ferrite -> 47uH; footprint (none) -> Inductor_SMD:L_Sagami_CER1257B; DPN (none) -> 308-2182-1-ND
- L2: value L_Ferrite -> 4.7uH; footprint (none) -> Inductor_SMD:L_Wuerth_HCM-1190; DPN (none) -> 732-1099-1-ND
Other:
- note removed: "600V"

Commit message: V0.3 schematic complete, footprints, 3d mods, prelim plancement. Ready for review then routing.
Parts:
- removed BT1: AAA Battery, Battery:BatteryHolder_Keystone_2466_1xAAA, symbol Device:Battery_Cell
- removed D2: BAV99, Package_TO_SOT_SMD:SOT-23, symbol Diode:BAV99
- removed J4: Conn_01x05, Connector_JST:CONN_B5B-ZR-SM4-TF_JST, symbol Connector_Generic:Conn_01x05
- removed J5: Screw_Terminal_01x03, TerminalBlock_TE-Connectivity:TerminalBlock_TE_282834-3_1x03_P2.54mm_Horizontal, symbol Connector:Screw_Terminal_01x03
- added C6: 1u, Capacitor_SMD:C_0603_1608Metric, symbol Device:C_Small
- added D2: CD0603-B0340R, Diode_SMD:D_0603_1608Metric, symbol Device:D_Schottky
- added J3: Screw_Terminal_01x04, TerminalBlock_TE-Connectivity:TerminalBlock_TE_282834-4_1x04_P2.54mm_Horizontal, symbol Connector:Screw_Terminal_01x04
- added R2, R6: 3K3, Resistor_SMD:R_0603_1608Metric, symbol Device:R
- L1: footprint Inductor_SMD:L_Sagami_CER1257B -> Inductor_SMD:L_1008_2520Metric; DPN 308-2182-1-ND -> 445-16442-1-ND
- L2: footprint Inductor_SMD:L_Wuerth_HCM-1190 -> Inductor_SMD:L_1210_3225Metric; DPN 732-1099-1-ND -> 587-1624-1-ND
- LS1: value Speaker -> Piezo; DPN (none) -> 2223-CPT-9019A-SMT-TRCT-ND
- Q1, Q2: DPN (none) -> SI2356DS-T1-GE3CT-ND
- R10: value 100K -> 147K
- R11: value 10K -> 6K34
- R12: value 100K -> 976K
- R13: value 10K -> 562K
- U2: DPN (none) -> MAX5026EUT+TCT-ND
- U3: value KXTJ3-1057 -> MXC4005XC; footprint Package_LGA:Kionix_LGA-12_2x2mm_P0.5mm_LayoutBorder2x4y -> Sensor:MXC4005XC_MEM-M; DPN (none) -> 1267-1075-1-ND
Connections:
- net adc_clk is gone; now on net deploy: J2.19 (Pin_19), U1.6 (GPIO15)
- net adc_miso is gone; now on net dump: J2.21 (Pin_21), U1.7 (GPIO16)
- net adc_mosi is gone; now on net charge: J2.23 (Pin_23), U1.8 (GPIO17)
- net adc_ncs is gone; now on net sw1: J2.25 (Pin_25), U1.9 (GPIO18)
- net fault_led is gone; now on net sda: J2.13 (Pin_13), U1.3 (GPIO12)
- net period is gone; now on net speaker+: J2.5 (Pin_5), U1.23 (GPIO8)
- net pump is gone; now on net speaker-: J2.7 (Pin_7), U1.24 (GPIO9)
- net setup is gone; now on net sw4: J1.6 (Pin_6), U1.20 (GPIO7)
- net start is gone; now on net sw3: J1.20 (Pin_20), U1.13 (GPIO0)
- net time_led is gone; now on net cont_en: J2.15 (Pin_15), U1.4 (GPIO13)
- net +3.3V: now also C3.1, C5.1, L1.1, Q7.2 (E), R12.2, R8.2, U2.5 (VCC), U3.6 (VDD), U4.5 (VOUT), C6.1, R2.2, R6.2
- net GND: now also C1.2, C3.2, C4.2, C5.2, Q1.2 (S), Q2.2 (S), Q6.2 (E), R11.1, R13.1, U2.1 (PGND), U2.2 (GND), U3.3 (GND), U4.2 (GND), C6.2, J3.2 (Pin_2)
- net sw2: now also J1.18 (Pin_18), U1.14 (GPIO1)
- net at R11.2: now also R10.1, U2.3 (FB)
- net +BATT: now reaches L2.1
- net +BATT: now also C4.1, U4.3 (EN), U4.6 (VIN), J3.1 (Pin_1)
- net at L2.2: now also U4.1 (SW)
- net at R7.1: now also Q6.1 (B)
- net at R7.2: now also Q2.3 (D), R3.1, J3.4 (Pin_4)
- net scl: now reaches U3.1 (SCL)
- net scl: now also J2.11 (Pin_11), U1.2 (GPIO11), R2.1
- net sda: now reaches U3.5 (SDA)
- net sda: now also R6.1
- net cont_sns: now reaches Q6.3 (C)
- net cont_sns: now also J2.17 (Pin_17), R8.1, U1.5 (GPIO14)
- net dump: now reaches Q1.1 (G)
- net cap_30v: now reaches Q1.3 (D)
- net cap_30v: now also C1.1, R10.2, D2.1 (K), J3.3 (Pin_3)
- net at U4.4 (VFB): now also R12.1, R13.2
- net deploy: now reaches Q2.1 (G)
- net at R14.1: now also Q7.1 (B)
- net cont_en: now reaches R14.2
- net at Q7.3 (C): now also R3.2
- net charge: now reaches U2.4 (EN)
- net at U2.6 (LX): now also L1.2, D2.2 (A)
- net speaker+: now reaches LS1.1
- net speaker-: now reaches LS1.2
- removed net run_led: D3.2 (A), J2.11 (Pin_11), U1.2 (GPIO11)
- net timeout renamed status_led
- net status_led: now also D3.2 (A)
Other:
- note added: "15mJ"
- note added: "3.3v Power"
- note added: "30V Deployment"
- note added: "Delay Time"
- note added: "Launch Deployment Timer"
- note added: "active low cont_en is only asserted when dump=1 is sunting the cap else damage to Q7 may occur with 30v present. A capacitor shunt across the cap by shorting pins 2&3 on the terminals, while still allowing continuity test."
- note removed: "Analog to Digital"
- note removed: "Connector / Protection"
- note removed: "FRONT PANEL"
- note removed: "LDT Launch Deployment timer"
- note removed: "Voltage Regs"
- moved on the sheet: C1, C10, C2, C3, C4, C5, C9, D3, J1, J2, L1, L2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

Commit message: Detailed BOM update, Stocked DPNs added. $16cad (or $26 with emulator connectors)
Parts:
- J1, J2: DPN ESW-113-12-T-D-ND -> SAM11102-ND
- J3: DPN (none) -> 732-691210910004-ND
- Q6: DPN (none) -> 4878-MMBT3904CT-ND
- Q7: DPN (none) -> 4878-MMBT3906CT-ND
- R10: DPN P100KHCT-ND -> P147KHCT-ND
- R11: DPN P10.0KHCT-ND -> P6.34KHCT-ND
- R12: DPN P100KHCT-ND -> P976KHCT-ND
- R13: DPN P10.0KHCT-ND -> P562KHCT-ND
- R2, R6: DPN P10.0KHCT-ND -> 311-3.30KHRCT-ND
- R9: value 3k3 -> 3K3
- SW1: DPN (none) -> 563-CFS-0400TACT-ND
- U4: DPN (none) -> MCP1640BT-I/CHYCT-ND
Changed lines of the file:
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@@
       (effects (font (size 1.27 1.27)) hide)
     )
-    (property "Datasheet" "~" (at 86.36 230.505 0)
+    (property "Datasheet" "" (at 86.36 230.505 0)
       (effects (font (size 1.27 1.27)) hide)
     )
@@
       (effects (font (size 1.27 1.27)) hide)
     )
-    (property "DPN" "P10.0KHCT-ND" (at 86.36 230.505 0)
+    (property "DPN" "P6.34KHCT-ND" (at 86.36 230.505 0)
       (effects (font (size 1.27 1.27)) hide)
     )
@@
       (effects (font (size 1.27 1.27)) hide)
     )
-    (property "Datasheet" "~" (at 145.415 125.73 0)
+    (property "Datasheet" "" (at 145.415 125.73 0)
       (effects (font (size 1.27 1.27)) hide)
     )
@@
       (effects (font (size 1.27 1.27)) hide)
     )
-    (property "DPN" "P10.0KHCT-ND" (at 145.415 125.73 0)
+    (property "DPN" "311-3.30KHRCT-ND" (at 145.415 125.73 0)
       (effects (font (size 1.27 1.27)) hide)
     )
@@
       (effects (font (size 1.27 1.27)) hide)
     )
-    (property "Datasheet" "https://jlcpcb.com/partdetail/Panasonic-ERJUP3F1002V/C491211" (at 168.91 224.79 0)
+    (property "Datasheet" "" (at 168.91 224.79 0)
       (effects (font (size 1.27 1.27)) hide)
     )
@@
       (effects (font (size 1.27 1.27) italic) (justify left) hide)
     )
-    (property "Datasheet" "https://www.onsemi.com/pub/Collateral/2N3903-D.PDF" (at 161.925 248.285 0)
+    (property "Datasheet" "https://www.digikey.ca/en/products/detail/diotec-semiconductor/MMBT3904/13163698" (at 161.925 248.285 0)
       (effects (font (size 1.27 1.27)) (justify left) hide)
     )
+    (property "DPN" "4878-MMBT3904CT-ND" (at 161.925 248.285 0)
+      (effects (font (size 1.27 1.27)) hide)
+    )
     (pin "1")
     (pin "2")
@@
       (effects (font (size 1.27 1.27)) hide)
     )
-    (property "Datasheet" "~" (at 159.385 237.49 0)
+    (property "Datasheet" "" (at 159.385 237.49 0)
       (effects (font (size 1.27 1.27)) hide)
     )
@@
       (effects (font (size 1.27 1.27)) hide)
     )
-    (property "Datasheet" "~" (at 120.65 187.325 0)
+    (property "Datasheet" "https://www.digikey.ca/en/products/detail/w%C3%BCrth-elektronik/691210910004/11477505" (at 120.65 187.325 0)
+      (effects (font (size 1.27 1.27)) hide)
+    )
+    (property "DPN" "732-691210910004-ND" (at 120.65 187.325 0)
       (effects (font (size 1.27 1.27)) hide)
     )
@@
       (effects (font (size 1.27 1.27)) hide)
     )
-    (property "Datasheet" "~" (at 339.725 208.915 0)
+    (property "Datasheet" "https://www.digikey.ca/en/products/detail/nidec-components/CFS-0400TA/12142605" (at 339.725 208.915 0)
+      (effects (font (size 1.27 1.27)) hide)
+    )
+    (property "DPN" "563-CFS-0400TACT-ND" (at 339.725 208.915 0)
       (effects (font (size 1.27 1.27)) hide)
     )
@@
       (effects (font (size 1.27 1.27) italic) (justify left) hide)
     )
-    (property "Datasheet" "http://ww1.microchip.com/downloads/en/DeviceDoc/20002234D.pdf" (at 344.17 57.785 0)
+    (property "Datasheet" "https://www.digikey.ca/en/products/detail/microchip-technology/MCP1640BT-I-CHY/2258563" (at 344.17 57.785 0)
+      (effects (font (size 1.27 1.27)) hide)
+    )
+    (property "DPN" "MCP1640BT-I/CHYCT-ND" (at 350.52 69.215 0)
       (effects (font (size 1.27 1.27)) hide)
     )
@@
       (effects (font (size 1.27 1.27)) hide)
     )
-    (property "Datasheet" "~" (at 137.795 125.73 0)
+    (property "Datasheet" "" (at 137.795 125.73 0)
       (effects (font (size 1.27 1.27)) hide)
     )
@@
       (effects (font (size 1.27 1.27)) hide)
     )
-    (property "DPN" "P10.0KHCT-ND" (at 137.795 125.73 0)
+    (property "DPN" "311-3.30KHRCT-ND" (at 137.795 125.73 0)
       (effects (font (size 1.27 1.27)) hide)
     )
@@
       (effects (font (size 1.27 1.27)) hide)
     )
-    (property "Datasheet" "https://jlcpcb.com/partdetail/Panasonic-ERJUP3F1002V/C491211" (at 86.36 219.075 0)
+    (property "Datasheet" "" (at 86.36 219.075 0)
       (effects (font (size 1.27 1.27)) hide)
     )
@@
       (effects (font (size 1.27 1.27)) hide)
     )
-    (property "DPN" "P100KHCT-ND" (at 86.36 219.075 0)
+    (property "DPN" "P147KHCT-ND" (at 86.36 219.075 0)
       (effects (font (size 1.27 1.27)) hide)
     )
@@
       (effects (font (size 1.27 1.27)) hide)
     )
-    (property "Datasheet" "~" (at 154.305 196.215 0)
+    (property "Datasheet" "" (at 154.305 196.215 0)
       (effects (font (size 1.27 1.27)) hide)
     )
@@
       (effects (font (size 1.27 1.27) italic) (justify left) hide)
     )
-    (property "Datasheet" "https://www.onsemi.com/pub/Collateral/2N3906-D.PDF" (at 166.37 196.215 0)
+    (property "Datasheet" "https://www.digikey.ca/en/products/detail/diotec-semiconductor/MMBT3906/13163222" (at 166.37 196.215 0)
       (effects (font (size 1.27 1.27)) (justify left) hide)
     )
+    (property "DPN" "4878-MMBT3906CT-ND" (at 166.37 196.215 0)
+      (effects (font (size 1.27 1.27)) hide)
+    )
     (pin "1")
     (pin "2")
@@
       (effects (font (size 1.27 1.27)) hide)
     )
-    (property "Datasheet" "https://jlcpcb.com/partdetail/Panasonic-ERJUP3F1002V/C491211" (at 370.205 72.39 0)
+    (property "Datasheet" "" (at 370.205 72.39 0)
       (effects (font (size 1.27 1.27)) hide)
     )
@@
       (effects (font (size 1.27 1.27)) hide)
     )
-    (property "DPN" "P100KHCT-ND" (at 370.205 72.39 0)
+    (property "DPN" "P976KHCT-ND" (at 370.205 72.39 0)
       (effects (font (size 1.27 1.27)) hide)
     )
@@
       (effects (font (size 1.27 1.27)) (justify right))
     )
-    (property "Value" "3k3" (at 90.17 48.895 0)
+    (property "Value" "3K3" (at 90.17 48.895 0)
       (effects (font (size 1.27 1.27)) (justify right))
     )
@@
       (effects (font (size 1.27 1.27)) hide)
     )
-    (property "Datasheet" "https://www.digikey.ca/en/products/detail/samtec-inc/ESW-113-12-T-D/7207386" (at 154.305 64.135 0)
-      (effects (font (size 1.27 1.27)) hide)
-    )
-    (property "DPN" "ESW-113-12-T-D-ND" (at 154.305 64.135 0)
+    (property "Datasheet" "https://www.digikey.ca/en/products/detail/samtec-inc/ESQ-113-13-L-D/6693822" (at 154.305 64.135 0)
+      (effects (font (size 1.27 1.27)) hide)
+    )
+    (property "DPN" "SAM11102-ND" (at 154.305 64.135 0)
       (effects (font (size 1.27 1.27)) hide)
     )
@@
       (effects (font (size 1.27 1.27)) hide)
     )
-    (property "Datasheet" "~" (at 370.205 83.185 0)
+    (property "Datasheet" "" (at 370.205 83.185 0)
       (effects (font (size 1.27 1.27)) hide)
     )
@@
       (effects (font (size 1.27 1.27)) hide)
     )
-    (property "DPN" "P10.0KHCT-ND" (at 370.205 83.185 0)
+    (property "DPN" "P562KHCT-ND" (at 370.205 83.185 0)
       (effects (font (size 1.27 1.27)) hide)
     )
@@
       (effects (font (size 1.27 1.27)) hide)
     )
-    (property "Datasheet" "https://www.digikey.ca/en/products/detail/samtec-inc/ESW-113-12-T-D/7207386" (at 69.215 64.135 0)
-      (effects (font (size 1.27 1.27)) hide)
-    )
-    (property "DPN" "ESW-113-12-T-D-ND" (at 69.215 64.135 0)
+    (property "Datasheet" "https://www.digikey.ca/en/products/detail/samtec-inc/ESQ-113-13-L-D/6693822" (at 69.215 64.135 0)
+      (effects (font (size 1.27 1.27)) hide)
+    )
+    (property "DPN" "SAM11102-ND" (at 69.215 64.135 0)
       (effects (font (size 1.27 1.27)) hide)
     )
@@
       (effects (font (size 1.27 1.27)) hide)
     )
-    (property "Datasheet" "~" (at 168.91 208.28 0)
-      (effects (font (size 1.27 1.27)) hide)
-    )
+    (property "Datasheet" "" (at 168.91 208.28 0)
+      (effects (font (size 1.27 1.27)) hide)
+    )

Commit message: Added Fram in soic-8 as flight recorder for validation flights
Parts:
- added U7: FM24W256, Package_SO:SOIC-8_3.9x4.9mm_P1.27mm, symbol Memory_NVRAM:FM24C64B
Connections:
- net +3.3V: now also U7.8 (VDD)
- net GND: now also U7.4 (VSS)
- net scl: now also U7.6 (SCL)
- net sda: now also U7.5 (SDA)
- no-connect marks 1 -> 8
Other:
- note added: "Fram"
- moved on the sheet: C6, R2, R6, U3

Commit message: pcb v0.5 added fram, and isp hdr, first place and route, assigned chip i/o to match routing.
Parts:
- added C7: 0.1u, Capacitor_SMD:C_0603_1608Metric, symbol Device:C_Small
- added J4: Conn_01x05, Connector_JST:CONN_B5B-ZR-SM4-TF_JST, symbol Connector_Generic:Conn_01x05
- added R15: 3K3, Resistor_SMD:R_0603_1608Metric, symbol Device:R
Connections:
- net +3.3V: now also C7.1, J4.1 (Pin_1), R15.2
- net GND: now also C7.2, J4.5 (Pin_5)
- net charge: now also J2.21 (Pin_21), U1.7 (GPIO16); no longer J2.23 (Pin_23), U1.8 (GPIO17)
- net cont_en: now also J2.17 (Pin_17), U1.5 (GPIO14); no longer J2.15 (Pin_15), U1.4 (GPIO13)
- net cont_sns: now also J2.19 (Pin_19), U1.6 (GPIO15); no longer J2.17 (Pin_17), U1.5 (GPIO14)
- net deploy: now also J1.18 (Pin_18), U1.14 (GPIO1); no longer J2.19 (Pin_19), U1.6 (GPIO15)
- net dump: now also J1.20 (Pin_20), U1.13 (GPIO0); no longer J2.21 (Pin_21), U1.7 (GPIO16)
- net reset_n: now also J4.4 (Pin_4), R15.1
- net scl: now also J2.23 (Pin_23), U1.8 (GPIO17), J4.2 (Pin_2); no longer J2.11 (Pin_11), U1.2 (GPIO11)
- net sda: now also J2.25 (Pin_25), U1.9 (GPIO18), J4.3 (Pin_3); no longer J2.13 (Pin_13), U1.3 (GPIO12)
- net speaker+: now also J2.13 (Pin_13), U1.3 (GPIO12); no longer J2.5 (Pin_5), U1.23 (GPIO8)
- net speaker-: now also J2.11 (Pin_11), U1.2 (GPIO11); no longer J2.7 (Pin_7), U1.24 (GPIO9)
- net sw1: now also J1.6 (Pin_6), U1.20 (GPIO7); no longer J2.25 (Pin_25), U1.9 (GPIO18)
- net sw2: now also J2.5 (Pin_5), U1.23 (GPIO8); no longer J1.18 (Pin_18), U1.14 (GPIO1)
- net sw3: now also J2.7 (Pin_7), U1.24 (GPIO9); no longer J1.20 (Pin_20), U1.13 (GPIO0)
- net sw4: now also J2.15 (Pin_15), U1.4 (GPIO13); no longer J1.6 (Pin_6), U1.20 (GPIO7)
- no-connect marks 8 -> 7
Other:
- note added: "+"
- note added: "2ohm"
- note added: "AAA battery"
- note added: "ISP"
- note added: "active low cont_en asserted if dump is asserted to hold capacitor voltage to zero."
- note added: "e"
- note added: "e-safe shunt"
- note added: "pull pin 4 (reset_n) low for external i2c fram read"
- note removed: "active low cont_en is only asserted when dump=1 is sunting the cap else damage to Q7 may occur with 30v present. A capacitor shunt across the cap by shorting pins 2&3 on the terminals, while still allowing continuity test."
- moved on the sheet: C1, C3, C6, D2, J3, L1, Q1, Q2, Q6, Q7, R10, R11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

Commit message: PCB v0.7 schem, pdf, pcb, gerbs
Parts:
- added C8: 0.1u, Capacitor_SMD:C_0603_1608Metric, symbol Device:C_Small
- added R16: dni, Resistor_SMD:R_0603_1608Metric, symbol Device:R
- added TP2: GND, TestPoint:TestPoint_Keystone_5000-5004_Miniature, symbol Connector:TestPoint
- added X1: ASE-48MHz, Oscillator:Oscillator_SMD_Abracon_ASV-4Pin_7.0x5.1mm_HandSoldering, symbol Oscillator:ASE-xxxMHz
Connections:
- net +3.3V: now also C8.1, X1.1 (EN), X1.4 (Vdd)
- net GND: now also C8.2, TP2.1, X1.2 (GND)
- net osc: now also R16.1
- net nc_nc: now reaches U3.2 (nc)
- net nc_int: now reaches U3.4 (INT)
- new net: R16.2, X1.3 (OUT)
- no-connect marks 7 -> 6
Other:
- moved on the sheet: C10, C2, C4, C5, C6, C9, D3, J1, J2, L2, LS1, R1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

Commit message: Update to v0.8 pcb, sch, bom, gerbs, pdf. Tapeout candidate?
Parts:
- added R23: dni, Resistor_SMD:R_0603_1608Metric, symbol Device:R
- added U5: AT25xxx, Package_SO:SOIC-8_3.9x4.9mm_P1.27mm, symbol Memory_EEPROM:AT25xxx
- added U8: LM809, Package_TO_SOT_SMD:SOT-23, symbol Power_Supervisor:LM809
- R16: DPN P22.0HCT-ND -> (none)
- R5: value DNI -> dni
Connections:
- net +3.3V: now also U5.8 (VCC), U8.3 (VCC)
- net GND: now also U5.4 (GND), U8.1 (GND)
- net reset_n: now also R23.1
- net spi_ck: now also U5.6 (SCK)
- net spi_si: now also U5.5 (MOSI)
- net spi_so: now also U5.2 (MISO)
- net spi_ss: now also U5.1 (~{CS})
- new net: R23.2, U8.2 (~{RESET})
- no-connect marks 6 -> 8
Other:
- note added: "Cut-away parts"
- note added: "Flight Recorder Opt."
- note added: "Front Panel"
- note removed: "Delay Time"
- note removed: "Fram"
- note removed: "ISP"
- note removed: "Piezo"
- moved on the sheet: C10, C2, C4, C5, C6, C8, C9, D3, J1, J2, L2, LS1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

Commit message: V0.9 pcb in progress.
Parts:
- added C11: 1u, Capacitor_SMD:C_0603_1608Metric, symbol Device:C_Small
- added D1: MM3Z12, Diode_SMD:D_SOD-323F, symbol Diode:MM3Zxx
- added Q3, Q5: MMBT3904, Package_TO_SOT_SMD:SOT-23, symbol Transistor_BJT:MMBT3904
- added Q4: SL2319, Package_TO_SOT_SMD:SOT-23, symbol Transistor_FET:AO3401A
- added Q8: SI2333, Package_TO_SOT_SMD:SOT-23, symbol Transistor_FET:AO3401A
- added R17: 1M, Resistor_SMD:R_0603_1608Metric, symbol Device:R
- added R18, R19, R20, R21, R22, R24, R25: 10K, Resistor_SMD:R_0603_1608Metric, symbol Device:R
- added R26: 100K, Resistor_SMD:R_0603_1608Metric, symbol Device:R
- L1: footprint Inductor_SMD:L_1008_2520Metric -> Inductor_SMD:L_1210_3225Metric; DPN 445-16442-1-ND -> 587-3069-1-ND
- R2, R6: value 3K3 -> 2K7; DPN 311-3.30KHRCT-ND -> 311-2.70KHRCT-ND
- R3: value 10K -> 1M; DPN P10.0KHCT-ND -> 311-1.00MHRCT-ND
- R7: value 100K -> 1M; DPN P100KHCT-ND -> 311-1.00MHRCT-ND
- R8: value 10K -> 100K; DPN P10.0KHCT-ND -> P100KHCT-ND
Connections:
- net +3.3V: now also R20.2
- net +BATT: now also Q8.3 (D); no longer C4.1, L2.1, U4.3 (EN), U4.6 (VIN)
- net GND: now also C11.2, Q3.2 (E), Q5.2 (E), R21.1, R22.1, R24.1, R26.1
- net cap_30v: now also Q4.3 (D); no longer D2.1 (K), R10.2
- net charge: now also R19.2, R24.2
- net cont_en: now also R25.2; no longer R14.2
- net deploy: now also R22.2
- net dump: now also R21.2
- new net: Q5.1 (B), R25.1
- new net: Q8.1 (G), R26.2
- new net: C4.1, L2.1, Q8.2 (S), U4.3 (EN), U4.6 (VIN)
- new net: Q5.3 (C), R14.2, R20.1
- new net: Q3.1 (B), R19.1
- new net: Q3.3 (C), R18.1
- new net: D1.2 (A), Q4.1 (G), R17.1, R18.2
- new net: C11.1, D1.1 (K), D2.1 (K), Q4.2 (S), R10.2, R17.2
Other:
- note added: "0.9v - 1.7v"
- note added: "E=15mJ"
- note removed: "15mJ"
- note removed: "active low cont_en asserted if dump is asserted to hold capacitor voltage to zero."
- moved on the sheet: C1, C3, D2, J3, L1, Q1, Q2, Q6, Q7, R10, R11, R14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
