File: pcb/dev_board.kicad_sch (KiCad schematic)
At the start: 67 parts, among them J1 Conn_02x13_Odd_Even, J2 Conn_02x13_Odd_Even, J3 Screw_Terminal_01x04, J4 Conn_01x05, Q1 Si2356DS, Q2 Si2356DS, Q3 MMBT3904, Q4 SL2319, Q5 MMBT3904, Q6 MMBT3904, Q7 MMBT3906, Q8 SI2333, SW1 SW_DIP_x04, U1 XS-LDT-01, U2 MAX5026, U3 MXC4005XC, U4 MCP1640BCH, U5 AT25xxx, U6 TLV74311, U7 FM24W256, U8 LM809, X1 ASE-48MHz

Commit message: V0.99 pcb dev board schem, pcb, bom, pcba
Parts:
- C10, C11, C2, C6, C9: LCSC PN (none) -> C15849
- C3, C4, C5: LCSC PN (none) -> C29823
- C7, C8: LCSC PN (none) -> C14663
- D1: LCSC PN (none) -> C19077460
- D2: LCSC PN (none) -> C3759853
- D3: value RUN -> LED; LCSC PN (none) -> C2899911
- J4: LCSC PN (none) -> C265440
- L1: LCSC PN (none) -> C250235
- L2: LCSC PN (none) -> C117731
- Q1, Q2: LCSC PN (none) -> C5182104
- Q3, Q5, Q6: LCSC PN (none) -> C7420353
- Q4: LCSC PN (none) -> C347478
- Q7: LCSC PN (none) -> C7420354
- Q8: LCSC PN (none) -> C2998060
- R1: JLC C491211 -> (none); LCSC PN (none) -> C21189
- R10: JLC C491211 -> (none); LCSC PN (none) -> C2998060
- R11: LCSC PN (none) -> C23087
- R12: JLC C491211 -> (none); LCSC PN (none) -> C2933270
- R13: LCSC PN (none) -> C2933238
- R14, R18, R19, R20, R21, R22, R24, R25: LCSC PN (none) -> C25804
- R15: LCSC PN (none) -> C22978
- R16, R23: JLC C319967 -> (none)
- R17, R7: JLC C491211 -> (none); LCSC PN (none) -> C22935
- R2, R6: LCSC PN (none) -> C13167
- R26, R8: LCSC PN (none) -> C25803
- R3: LCSC PN (none) -> C22935
- R4: JLC C319967 -> (none); LCSC PN (none) -> C21190
- R5: JLC C491211 -> (none)
- R9: JLC C319967 -> (none); LCSC PN (none) -> C22978
- U2: LCSC PN (none) -> C87603
- U3: LCSC PN (none) -> C404327
- U4: LCSC PN (none) -> C478087
- U6: LCSC PN (none) -> C485147
- U7: LCSC PN (none) -> C66020

Commit message: Fixup LSCS part  num
Parts:
- Q8: LCSC PN C2998060 -> C344008
Changed lines of the file:
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@@
       (effects (font (size 1.27 1.27)) hide)
     )
-    (property "LCSC PN" "C2998060" (at 304.165 53.975 0)
+    (property "LCSC PN" "C344008" (at 304.165 53.975 0)
       (effects (font (size 1.27 1.27)) hide)
     )
