File: pcb/dev_board.kicad_pcb (KiCad board)
At the start: 6 copper layers, 45.7 x 50 mm, 52 parts, among them J1 Conn_02x13_Odd_Even, J2 Conn_02x13_Odd_Even, J3 Screw_Terminal_01x04, J4 Conn_01x05, Q1 Si2356DS, Q2 Si2356DS, Q6 MMBT3904, Q7 MMBT3906, SW1 SW_DIP_x04, U1 XS-LDT-01, U2 MAX5026, U3 MXC4005XC, U4 MCP1640BCH, U5 AT25xxx, U6 TLV74311, U7 FM24W256, U8 LM809, X1 ASE-48MHz

Commit message: V0.9 pcb in progress.
Parts:
- added C11: 1u, Capacitor_SMD:C_0603_1608Metric, B.Cu at (173.3, 111.4)
- added D1: MM3Z12, Diode_SMD:D_SOD-323F, B.Cu at (175.0, 116.1)
- added Q3: MMBT3904, Package_TO_SOT_SMD:SOT-23, B.Cu at (175.3, 120.4)
- added Q4: SL2319, Package_TO_SOT_SMD:SOT-23, B.Cu at (171.9, 120.4)
- added Q5: MMBT3904, Package_TO_SOT_SMD:SOT-23, B.Cu at (168.4, 120.4)
- added Q8: SI2333, Package_TO_SOT_SMD:SOT-23, B.Cu at (164.5, 99.6)
- added R17: 1M, Resistor_SMD:R_0603_1608Metric, B.Cu at (176.4, 112.5)
- added R18: 10K, Resistor_SMD:R_0603_1608Metric, B.Cu at (176.4, 116.1)
- added R19: 10K, Resistor_SMD:R_0603_1608Metric, B.Cu at (164.1, 106.5)
- added R20: 10K, Resistor_SMD:R_0603_1608Metric, B.Cu at (165.1, 121.5)
- added R21: 10K, Resistor_SMD:R_0603_1608Metric, B.Cu at (176.0, 106.4)
- added R22: 10K, Resistor_SMD:R_0603_1608Metric, B.Cu at (176.0, 103.1)
- added R24: 10K, Resistor_SMD:R_0603_1608Metric, B.Cu at (164.0, 103.2)
- added R25: 10K, Resistor_SMD:R_0603_1608Metric, B.Cu at (165.1, 119.5)
- added R26: 100K, Resistor_SMD:R_0603_1608Metric, B.Cu at (164.1, 95.0)
- R2, R6: value 3K3 -> 2K7
- R3: value 10K -> 1M
- R5: value DNI -> dni
- R7: value 100K -> 1M
- R8: value 10K -> 100K
- moved J3 4.22 mm to (166.4, 127.8)
- moved Q1 4.22 mm to (171.9, 124.2)
- moved Q2 4.22 mm to (175.4, 124.2)
- moved Q7 4.22 mm to (168.5, 124.2)
- moved R3 4.22 mm to (171.9, 130.1)
- moved R8 4.22 mm to (165.6, 130.1)
- moved Q6 4.22 mm to (165.1, 124.2)
- moved R14 4.22 mm to (168.8, 130.1)
- moved R7 4.22 mm to (175.1, 130.1)
- moved D3 3.61 mm to (175.8, 81.0), turned to -90 degrees
- moved C1 2.18 mm to (169.7, 118.4)
- moved C7 1.14 mm to (165.6, 95.0)
Connections:
- C4 pad 1: +BATT -> Net-(Q8-S)
- D2 pad 1: /cap_30v -> Net-(D1-K)
- L2 pad 1: +BATT -> Net-(Q8-S)
- R10 pad 2: /cap_30v -> Net-(D1-K)
- R14 pad 2: /cont_en -> Net-(Q5-C)
- U4 pad 3: +BATT -> Net-(Q8-S)
- U4 pad 6: +BATT -> Net-(Q8-S)
Routing:
- net Net-(Q8-S): track 0.00 -> 54.7 mm, vias 0 -> 2
- net +BATT: track 58.8 -> 6.28 mm, vias 2 -> 0
- net Net-(D1-K): track 0.00 -> 8.30 mm
- net Net-(D3-K): track 2.40 -> 10.3 mm
- net /cap_30v: track 20.9 -> 14.1 mm
- net Net-(Q5-C): track 0.00 -> 5.18 mm
- net /cont_en: track 46.2 -> 41.0 mm
- net /status_led: track 46.7 -> 48.5 mm
- net GND: track 62.1 -> 63.3 mm
Other:
- board size 45.7 x 50 mm -> 45.7 x 53.3 mm
- board text added: "+"
- board text added: "+1"
- board text added: "+bat-"
- board text added: "+out-"
- board text added: "-"
- board text added: "0.9v to 1.7v"
- board text added: "bat"
- board text removed: "+Bat-"
- board text removed: "+Out-"
- board text removed: "0.9v - 1.7v"

Commit message: V0.99 pcb dev board schem, pcb, bom, pcba
Parts:
- D3: value RUN -> LED
- L1: footprint Inductor_SMD:L_1008_2520Metric -> Inductor_SMD:L_1210_3225Metric
- moved R22 24.6 mm to (176.1, 127.8), turned to 90 degrees
- moved R19 12.1 mm to (165.2, 118.5), turned to 180 degrees
- moved C7 9.71 mm to (174.2, 99.4), turned to 180 degrees
- moved R24 5.96 mm to (165.5, 109.0), turned to 0 degrees
- moved R21 3.59 mm to (174.1, 109.5), turned to 0 degrees
- moved D3 3.43 mm to (175.6, 84.5)
- moved R18 3.25 mm to (174.9, 113.3), turned to 90 degrees
- moved Q8 2.89 mm to (165.7, 97.0), turned to -90 degrees
- moved R17 2.73 mm to (174.1, 111.0), turned to 180 degrees
- moved R2 2.30 mm to (176.0, 96.1)
- moved R6 2.30 mm to (176.0, 93.1), turned to 90 degrees
- moved R26 1.53 mm to (164.7, 93.6), turned to -90 degrees
- moved C11 1.28 mm to (172.6, 112.5), turned to 180 degrees
- moved U7 1.25 mm to (171.4, 95.9)
- moved LS1 0.95 mm to (169.2, 84.7)
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Routing:
- net Net-(Q8-S): track 54.7 -> 21.9 mm, vias 2 -> 0
- net +BATT: track 6.28 -> 33.1 mm, vias 0 -> 2
- net Net-(Q3-B): track 0.00 -> 23.3 mm
- net GND: track 63.3 -> 78.7 mm, vias 29 -> 31
- net Net-(D1-A): track 0.00 -> 12.8 mm
- net Net-(Q5-C): track 5.18 -> 17.6 mm
- net /cont_sns: track 42.2 -> 54.0 mm
- net Net-(D1-K): track 8.30 -> 16.5 mm
- net /deploy: track 35.7 -> 42.8 mm
- net /dump: track 36.6 -> 43.6 mm
- net Net-(Q3-C): track 0.00 -> 6.12 mm
- net Net-(D3-K): track 10.3 -> 4.36 mm
- net /cont_en: track 41.0 -> 36.0 mm
- net /charge: track 34.8 -> 38.9 mm
- net Net-(Q5-B): track 0.00 -> 3.85 mm
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