File: pcb/prod_board.kicad_pcb (KiCad board)
At the start: 4 copper layers, 14.2 x 53.3 mm, 60 parts, among them J3 TE_282834-4, J4 B5B-ZR-SM4-TF, Q1 Si2356DS, Q2 Si2356DS, Q3 MMBT3904, Q4 SL2319, Q5 MMBT3904, Q6 MMBT3904, Q7 MMBT3906, Q8 SI2333, SW1 CFS-0400TA, U1 XS-LDT-01, U2 MAX5026, U3 MXC4005XC, U4 MCP1640BCH, U6 TLV74311, U7 FM24W256

Commit message: Pcb PB updated to fix missing net
Routing:
- net /sda: track 46.6 -> 47.7 mm
Changed lines of the file:
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@@
     (title "XS-LDT-PB Product Board")
     (date "2026-09-23")
-    (rev "V1")
+    (rev "V1.1")
     (company "Eric Pearson: XYZZY Semiconductor")
   )
@@
     (pts (xy 163.068 78.74) (xy 163.068 132.08))
     (height 11.811)
-    (gr_text "2100.0000 mils" (at 150.107 105.41 90) (layer "Dwgs.User")
+    (gr_text "53.3400 mm" (at 150.107 105.41 90) (layer "Dwgs.User")
       (effects (font (size 1 1) (thickness 0.15)))
     )
@@
     (pts (xy 163.068 78.6662) (xy 177.292 78.6662))
     (height -7.0382)
-    (gr_text "560.0000 mils" (at 170.18 70.478) (layer "Dwgs.User")
+    (gr_text "14.2240 mm" (at 170.18 70.478) (layer "Dwgs.User")
       (effects (font (size 1 1) (thickness 0.15)))
     )
@@
   (via (at 169.49 109.264737) (size 0.6) (drill 0.35) (layers "F.Cu" "B.Cu") (net 17))
   (via (at 175.2346 93.218) (size 0.6) (drill 0.35) (layers "F.Cu" "B.Cu") (net 17))
+  (segment (start 175.2346 93.218) (end 175.324 93.218) (width 0.127) (layer "B.Cu") (net 17))
   (segment (start 169.8244 111.0996) (end 171.3992 111.0996) (width 0.127) (layer "B.Cu") (net 17))
+  (segment (start 175.324 93.218) (end 176.022 93.916) (width 0.127) (layer "B.Cu") (net 17))
   (segment (start 170.1292 83.1596) (end 170.1292 81.1995) (width 0.127) (layer "B.Cu") (net 17))
   (segment (start 170.3324 83.3628) (end 170.1292 83.1596) (width 0.127) (layer "B.Cu") (net 17))
